Commit message: update with 23 DOF x1

File: humanoidverse/data/robots/x1/xyber_x1_serial.urdf (robot description, URDF)
Before this commit: robot x1, 58 links, 57 joints
Joints:
- joint left_elbow_pitch_joint: limit lower=-3.14 upper=3.14 effort=0 velocity=0 -> lower=-3.14 upper=3.14 effort=150 velocity=8; type fixed -> revolute
- joint left_shoulder_roll_joint: limit lower=-3.14 upper=3.14 effort=0 velocity=0 -> lower=-3.14 upper=3.14 effort=150 velocity=8; type fixed -> revolute
- joint left_shoulder_yaw_joint: limit lower=-3.14 upper=3.14 effort=0 velocity=0 -> lower=-3.14 upper=3.14 effort=150 velocity=8; type fixed -> revolute
- joint lumber_pitch_joint: limit lower=-3.14 upper=3.14 effort=0 velocity=0 -> lower=-3.14 upper=3.14 effort=50 velocity=37; type fixed -> revolute
- joint lumber_roll_joint: limit lower=-3.14 upper=3.14 effort=0 velocity=0 -> lower=-3.14 upper=3.14 effort=50 velocity=37; type fixed -> revolute
- joint lumber_yaw_joint: limit lower=-3.14 upper=3.14 effort=0 velocity=0 -> lower=-3.14 upper=3.14 effort=88 velocity=32; type fixed -> revolute
- joint right_elbow_pitch_joint: limit lower=-3.14 upper=3.14 effort=0 velocity=0 -> lower=-3.14 upper=3.14 effort=150 velocity=8; type fixed -> revolute
- joint right_shoulder_roll_joint: limit lower=-3.14 upper=3.14 effort=0 velocity=0 -> lower=-3.14 upper=3.14 effort=150 velocity=8; type fixed -> revolute
- joint right_shoulder_yaw_joint: limit lower=-3.14 upper=3.14 effort=0 velocity=0 -> lower=-3.14 upper=3.14 effort=150 velocity=8; type fixed -> revolute
